File: eagle/match_best.sch (EAGLE design)
At the start: 7 parts, among them X1 SMA-142-0711-821/826

Commit message: asdfg
Parts:
- L1: value DRR1,5A -> B82111; device inductors:DRR1,5A -> inductors:B82111
Changed lines of the file:
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@@
 <part name="TP2" library="testpad" deviceset="TP" device="PAD1-13Y"/>
 <part name="TP4" library="testpad" deviceset="TP" device="PAD1-13Y"/>
-<part name="L1" library="inductors" deviceset="DRR1,5A" device=""/>
+<part name="L1" library="inductors" deviceset="B82111" device=""/>
 <part name="C2" library="sprague" deviceset="C-TRIMM" device="" value="10-30"/>
 <part name="C5" library="resistor" deviceset="C-US" device="" value="100p"/>
